File: pcb/Board43.kicad_pcb (KiCad board)
At the start: 2 copper layers, 54 x 85.6 mm, 583 parts, among them J1 BM03B-SRSS-TB, J2 Conn_01x10_Pin, Q1 S9013, SW1 SW_Push, SW2 SW_Push, SW3 SW_Push, SW4 SW_Push, SW5 SW_Push, SW6 SW_Push, U1 LM73100RPWR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

Commit message: refactor: add PCB licenses
Rename symbol and footprint libraries from Board43 to Board43_KiCad
to clarify they are project-specific KiCad libraries. Update library
tables, schematic, and PCB references accordingly.

Add CERN-OHL-W-2.0 and CC-BY-SA-4.0 license files for the PCB design.
Parts:
- C18, C19: footprint Board43:C_0402_1005Metric_Narrow -> Board43_KiCad:C_0402_1005Metric_Narrow
- D2: footprint Board43:KT-0603W -> Board43_KiCad:KT-0603W
- U1: footprint Board43:LM73100RPWR -> Board43_KiCad:LM73100RPWR
- U3: footprint Board43:RP2350A -> Board43_KiCad:RP2350A
- U7: footprint Board43:TPD2EUSB30ADRTR -> Board43_KiCad:TPD2EUSB30ADRTR
Changed lines of the file:
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@@
 	(net 331 "unconnected-(USB1-SBU1-PadA8)")
 	(net 332 "unconnected-(USB1-SBU2-PadB8)")
+	(net 333 "unconnected-(U1-PGTH-Pad4)_1")
+	(net 334 "unconnected-(U1-DNC-Pad10)")
 	(footprint "Capacitor_SMD:C_0201_0603Metric"
 		(layer "F.Cu")
@@
 		)
 	)
-	(footprint "Board43:RP2350A"
+	(footprint "Board43_KiCad:RP2350A"
 		(layer "F.Cu")
 		(at 42.95 91.71 90)
@@
 			(at 0 5.2 90)
 			(layer "F.Fab")
-			(hide yes)
 			(effects
 				(font
@@
 			(pinfunction "GND")
 			(pintype "power_in")
+			(zone_connect 2)
 		)
 		(pad "61" thru_hole circle
@@
 			(pinfunction "GND")
 			(pintype "power_in")
+			(zone_connect 2)
 		)
 		(pad "61" thru_hole circle
@@
 			(pinfunction "GND")
 			(pintype "power_in")
+			(zone_connect 2)
 		)
 		(pad "61" thru_hole circle
@@
 			(pinfunction "GND")
 			(pintype "power_in")
+			(zone_connect 2)
 		)
 		(pad "61" thru_hole circle
@@
 			(pinfunction "GND")
 			(pintype "power_in")
+			(zone_connect 2)
 		)
 		(pad "61" smd roundrect
@@
 			(pinfunction "GND")
 			(pintype "power_in")
+			(zone_connect 2)
 		)
 		(pad "61" thru_hole circle
@@
 			(pinfunction "GND")
 			(pintype "power_in")
+			(zone_connect 2)
 		)
 		(pad "61" thru_hole circle
@@
 			(pinfunction "GND")
 			(pintype "power_in")
+			(zone_connect 2)
 		)
 		(pad "61" thru_hole circle
@@
 			(pinfunction "GND")
 			(pintype "power_in")
+			(zone_connect 2)
 		)
 		(embedded_fonts no)
@@
 		)
 	)
-	(footprint "Board43:LM73100RPWR"
+	(footprint "Board43_KiCad:LM73100RPWR"
 		(layer "F.Cu")
 		(at 22.03 93.825 180)
 		(property "Reference" "U1"
-			(at 0 -2.75 0)
+			(at 0 -2.75 180)
 			(layer "F.SilkS")
 			(hide yes)
@@
 		)
 		(property "Value" "LM73100RPWR"
-			(at 0 2.75 0)
+			(at 0 2.75 180)
 			(layer "F.Fab")
-			(hide yes)
 			(effects
 				(font
@@
 		)
 		(property "Datasheet" "https://www.lcsc.com/datasheet/C3210761.pdf"
-			(at 0 0 0)
+			(at 0 0 180)
 			(layer "F.Fab")
 			(hide yes)
@@
 		)
 		(property "Description" ""
-			(at 0 0 0)
+			(at 0 0 180)
 			(layer "F.Fab")
 			(hide yes)
@@
 		)
 		(fp_text user "${REFERENCE}"
-			(at 0 0 0)
+			(at 0 0 180)
 			(layer "F.Fab")
 			(effects
@@
 			(layers "F.Cu" "F.Mask" "F.Paste")
 			(roundrect_rratio 0.2)
-			(net 304 "unconnected-(U1-PGTH-Pad4)")
+			(net 333 "unconnected-(U1-PGTH-Pad4)_1")
 			(pinfunction "PGTH")
 			(pintype "input+no_connect")
@@
 			(layers "F.Cu" "F.Mask" "F.Paste")
 			(roundrect_rratio 0.2)
-			(net 303 "unconnected-(U1-DNC-Pad10)_1")
+			(net 334 "unconnected-(U1-DNC-Pad10)")
 			(pinfunction "DNC")
 			(pintype "no_connect")
@@
 		)
 	)
-	(footprint "Board43:KT-0603W"
+	(footprint "Board43_KiCad:KT-0603W"
 		(layer "F.Cu")
 		(at 28 84.15 75)
@@
 			(unlocked yes)
 			(layer "F.Fab")
-			(hide yes)
 			(effects
 				(font
@@
 		)
 	)
-	(footprint "Board43:C_0402_1005Metric_Narrow"
+	(footprint "Board43_KiCad:C_0402_1005Metric_Narrow"
 		(layer "F.Cu")
 		(at 38.29 89.71 90)
@@
 			(unlocked yes)
 			(layer "F.Fab")
-			(hide yes)
 			(effects
 				(font
@@
 		)
 	)
-	(footprint "Board43:C_0402_1005Metric_Narrow"
+	(footprint "Board43_KiCad:C_0402_1005Metric_Narrow"
 		(layer "F.Cu")
 		(at 37.35 89.71 90)
@@
 			(unlocked yes)
 			(layer "F.Fab")
-			(hide yes)
 			(effects
 				(font
@@
 		)
 	)
-	(footprint "Board43:TPD2EUSB30ADRTR"
+	(footprint "Board43_KiCad:TPD2EUSB30ADRTR"
 		(layer "F.Cu")
 		(at 28.09 96.18 90)
