File: pcb/Board43.kicad_sch (KiCad schematic)
At the start: 70 parts, among them J1 BM03B-SRSS-TB, J2 Conn_01x10_Pin, Q1 S9013, SW1 SW_Push, SW2 SW_Push, SW3 SW_Push, SW4 SW_Push, SW5 SW_Push, SW6 SW_Push, U1 LM73100RPWR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

Commit message: refactor: add PCB licenses
Rename symbol and footprint libraries from Board43 to Board43_KiCad
to clarify they are project-specific KiCad libraries. Update library
tables, schematic, and PCB references accordingly.

Add CERN-OHL-W-2.0 and CC-BY-SA-4.0 license files for the PCB design.
Parts:
- C18, C19: footprint Board43:C_0402_1005Metric_Narrow -> Board43_KiCad:C_0402_1005Metric_Narrow
- D2: footprint Board43:KT-0603W -> Board43_KiCad:KT-0603W
- L2: symbol Board43:AOTA-B201610S3R3-101-T -> Board43_KiCad:AOTA-B201610S3R3-101-T
- U1: footprint Board43:LM73100RPWR -> Board43_KiCad:LM73100RPWR
- U3: footprint Board43:RP2350A -> Board43_KiCad:RP2350A
- U7: footprint Board43:TPD2EUSB30ADRTR -> Board43_KiCad:TPD2EUSB30ADRTR
Changed lines of the file:
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@@
 	)
 	(symbol
-		(lib_id "Board43:AOTA-B201610S3R3-101-T")
+		(lib_id "Board43_KiCad:AOTA-B201610S3R3-101-T")
 		(at 195.58 62.23 90)
 		(unit 1)
@@
 			)
 		)
-		(property "Footprint" "Board43:C_0402_1005Metric_Narrow"
+		(property "Footprint" "Board43_KiCad:C_0402_1005Metric_Narrow"
 			(at 185.1152 67.31 0)
 			(effects
@@
 			)
 		)
-		(property "Footprint" "Board43:RP2350A"
+		(property "Footprint" "Board43_KiCad:RP2350A"
 			(at 243.84 149.86 0)
 			(effects
@@
 			)
 		)
-		(property "Footprint" "Board43:TPD2EUSB30ADRTR"
+		(property "Footprint" "Board43_KiCad:TPD2EUSB30ADRTR"
 			(at 185.42 275.59 0)
 			(effects
@@
 			)
 		)
-		(property "Footprint" "Board43:C_0402_1005Metric_Narrow"
+		(property "Footprint" "Board43_KiCad:C_0402_1005Metric_Narrow"
 			(at 173.6852 67.31 0)
 			(effects
@@
 			)
 		)
-		(property "Footprint" "Board43:KT-0603W"
+		(property "Footprint" "Board43_KiCad:KT-0603W"
 			(at 293.37 114.3 0)
 			(effects
@@
 			)
 		)
-		(property "Footprint" "Board43:LM73100RPWR"
+		(property "Footprint" "Board43_KiCad:LM73100RPWR"
 			(at 140.97 58.42 0)
 			(effects
